File: hw/PCBs/Top_Board/Top_Board/Top_Board_Boundary_Ref.brd (EAGLE design)
At the start: 78 x 78 mm, 0 parts

Commit message: better readme
Parts:
- added C1, C2, C3, R1, R2, R3, R4, R5: (no value), SparkFun-Passives:0805
- added D1: (no value), SparkFun-DiscreteSemi:SMA-DIODE
- added D2: MBRA140, SparkFun-DiscreteSemi:SMA-DIODE
- added J1: (no value), SparkFun-Connectors:JST-2-SMD
- added L1: 27uH, SparkFun-Passives:INDUCTOR_SDR1307
- added U1: LT3652, SparkFun-PowerIC:MSOP-12_GND
Connections:
- new net GND: C2.2, C3.2, D2.A, J1.1, R3.1, R5.1, U1.13, U1.6
- new net N$1: R4.1, R5.2, U1.7
- new net N$2: C3.1, D1.A, J1.2, R1.1, R4.2, U1.9
- new net N$3: C1.1, D2.C, L1.P$1, U1.12
- new net N$4: C2.1, R2.2, U1.1, U1.3
- new net N$5: R2.1, R3.2, U1.2
- new net N$6: C1.2, D1.C, U1.11
- new net N$8: L1.P$2, R1.2, U1.10
